Commit message: update: add realsense urdf from realsense_ros, minor debugs

File: ur_elpis_control/urdf/my_robot_cell_controlled.urdf.xacro (robot description, xacro)
@@ -33,5 +33,5 @@
     visual_parameters_file="$(arg visual_params)"
   >
-    <origin xyz="0 0 1" rpy="0 0 0" />
+    <origin xyz="0 0 0" rpy="0 0 0" />
   </xacro:my_robot_cell>
   <!--Create the control tag for the UR robot-->
@@ -48,4 +48,24 @@
     headless_mode="$(arg headless_mode)"
   />
-  <!--If you had more controlled devices in your description, e.g. a gripper, you can add another ros2_control tag here-->
+  <!--Gripper ros2_control configuration-->
+  <!-- Note: Gripper control is currently handled via the /control_gripper service.
+       To enable ros2_control for the gripper, a custom hardware interface plugin
+       that wraps the gripper library (librh_p12_rna.so) would need to be created.
+       For now, the gripper joints are defined as revolute in the URDF for visualization
+       but are controlled via the service interface. -->
+  <!--
+  <ros2_control name="gripper" type="actuator">
+    <hardware>
+      <plugin>gripper_hardware/GripperHardwareInterface</plugin>
+    </hardware>
+    <joint name="rh_p12_rn">
+      <command_interface name="position">
+        <param name="min">0.0</param>
+        <param name="max">1.12</param>
+      </command_interface>
+      <state_interface name="position"/>
+      <state_interface name="velocity"/>
+    </joint>
+  </ros2_control>
+  -->
 </robot>

File: ur_elpis_description/urdf/my_robot_cell.urdf.xacro (robot description, xacro)
@@ -17,5 +17,5 @@
     visual_parameters_file="$(arg visual_parameters_file)"
     >
-      <origin xyz="0 0 1" rpy="0 0 0" />
+      <origin xyz="0 0 0" rpy="0 0 0" />
   </xacro:my_robot_cell>
 </robot>

File: ur_elpis_description/urdf/my_robot_cell_macro.xacro (robot description, xacro)
@@ -2,4 +2,5 @@
 <robot xmlns:xacro="http://ros.org/wiki/xacro">
   <xacro:include filename="$(find ur_description)/urdf/ur_macro.xacro"/>
+  <xacro:include filename="$(find realsense2_description)/urdf/_d435.urdf.xacro"/>
   <xacro:macro name="my_robot_cell" params="
     parent
@@ -123,5 +124,5 @@
     </material>
     <joint name="tool0_rh_p12_rn_base" type="fixed">
-      <origin rpy="0 0 -1.570796" xyz="0 0 0"/>
+      <origin rpy="0 0 1.570794" xyz="0 0 0"/>
       <parent link="${ur_type}_tool0"/>
       <child link="rh_p12_rn_base"/>
@@ -147,8 +148,10 @@
       </inertial>
     </link>
-    <joint name="rh_p12_rn" type="fixed">
+    <joint name="rh_p12_rn" type="revolute">
       <parent link="rh_p12_rn_base"/>
       <child link="rh_p12_rn_r1"/>
       <origin xyz="0.0 0.008 0.058" rpy="0 0 0"/>
+      <axis xyz="1 0 0"/>
+      <limit lower="0.0" upper="1.12" effort="100.0" velocity="1.0"/>
     </joint>
     <link name="rh_p12_rn_r1">
@@ -172,8 +175,11 @@
       </inertial>
     </link>
-    <joint name="rh_r2" type="fixed">
+    <joint name="rh_r2" type="revolute">
       <parent link="rh_p12_rn_r1"/>
       <child link="rh_p12_rn_r2"/>
       <origin xyz="0.0 0.0493634 0.0285" rpy="0 0 0"/>
+      <axis xyz="-1 0 0"/>
+      <limit lower="0.0" upper="1.12" effort="100.0" velocity="1.0"/>
+      <mimic joint="rh_p12_rn" multiplier="1.0" offset="0.0"/>
     </joint>
     <link name="rh_p12_rn_r2">
@@ -197,8 +203,11 @@
       </inertial>
     </link>
-    <joint name="rh_l1" type="fixed">
+    <joint name="rh_l1" type="revolute">
       <parent link="rh_p12_rn_base"/>
       <child link="rh_p12_rn_l1"/>
       <origin xyz="0.0 -0.008 0.058" rpy="0 0 0"/>
+      <axis xyz="-1 0 0"/>
+      <limit lower="0.0" upper="1.12" effort="100.0" velocity="1.0"/>
+      <mimic joint="rh_p12_rn" multiplier="1.0" offset="0.0"/>
     </joint>
     <link name="rh_p12_rn_l1">
@@ -222,8 +231,11 @@
       </inertial>
     </link>
-    <joint name="rh_l2" type="fixed">
+    <joint name="rh_l2" type="revolute">
       <parent link="rh_p12_rn_l1"/>
       <child link="rh_p12_rn_l2"/>
       <origin xyz="0.0 -0.0493634 0.0285" rpy="0 0 0"/>
+      <axis xyz="1 0 0"/>
+      <limit lower="0.0" upper="1.12" effort="100.0" velocity="1.0"/>
+      <mimic joint="rh_p12_rn" multiplier="1.0" offset="0.0"/>
     </joint>
     <link name="rh_p12_rn_l2">
@@ -262,4 +274,15 @@
     <!-- Camera (RealSense D435) -->
     <!-- ============================================ -->
+    <!-- Using realsense2_description macro for D435 camera -->
+    <!-- Camera transformation from tool0 to camera_color_frame (measured):
+         Matrix:
+         0.99825    -0.027368   -0.052507   -0.007395
+         0.028123    0.99951     0.013702   -0.051154
+         0.052107   -0.015155    0.99853     0.069229
+         0           0           0           1
+         Translation: x=-0.007395, y=-0.051154, z=0.069229
+         Rotation (RPY): roll=-0.01517, pitch=-0.05212, yaw=0.02815
+    -->
+    <!-- Old manual camera definition (commented out):
     <material name="white">
       <color rgba="1.0 1.0 1.0 1.0"/>
@@ -270,60 +293,29 @@
       <child link="d435_bottom_screw_frame"/>
     </joint>
-    <link name="d435_bottom_screw_frame">
-      <inertial>
-        <origin rpy="0 0 0" xyz="0 0 0"/>
-        <mass value="0.001"/>
-        <inertia ixx="1E-5" ixy="0" ixz="0" iyy="1E-5" iyz="-0" izz="1E-5"/>
-      </inertial>
-    </link>
-    <joint name="d435_link_joint" type="fixed">
-      <origin rpy="0 0 0" xyz="0 0.0175 0.0125"/>
-      <parent link="d435_bottom_screw_frame"/>
-      <child link="d435_link"/>
-    </joint>
-    <link name="d435_link">
-      <visual>
-        <origin rpy="1.5707963267948966 0 1.5707963267948966" xyz="0.0149 -0.0175 0"/>
-        <geometry>
-          <mesh filename="package://ur_elpis_description/assets/realsense2/visual/d435.obj"/>
-        </geometry>
-        <material name="white"/>
-      </visual>
-      <collision>
-        <origin rpy="0 0 0" xyz="0 -0.0175 0"/>
-        <geometry>
-          <box size="0.02505 0.09 0.025"/>
-        </geometry>
-      </collision>
-      <inertial>
-        <mass value="0.564"/>
-        <origin xyz="0 0 0"/>
-        <inertia ixx="0.003881243" ixy="0.0" ixz="0.0" iyy="0.000498940" iyz="0.0" izz="0.003879257"/>
-      </inertial>
-    </link>
-    <joint name="d435_depth_joint" type="fixed">
-      <origin rpy="1.5707963267948966 0 1.5707963267948966" xyz="0 0 0"/>
-      <parent link="d435_link"/>
-      <child link="d435_depth_frame"/>
-    </joint>
-    <link name="d435_depth_frame">
-      <inertial>
-        <origin rpy="0 0 0" xyz="0 0 0"/>
-        <mass value="0.001"/>
-        <inertia ixx="1E-5" ixy="0" ixz="0" iyy="1E-5" iyz="-0" izz="1E-5"/>
-      </inertial>
-    </link>
-    <joint name="d435_color_joint" type="fixed">
-      <origin rpy="0 0 0" xyz="-0.015 0 0"/>
-      <parent link="d435_depth_frame"/>
-      <child link="d435_color_frame"/>
-    </joint>
-    <link name="d435_color_frame">
-      <inertial>
-        <origin rpy="0 0 0" xyz="0 0 0"/>
-        <mass value="0.001"/>
-        <inertia ixx="1E-5" ixy="0" ixz="0" iyy="1E-5" iyz="-0" izz="1E-5"/>
-      </inertial>
-    </link>
+    ... (all the manual camera links and joints)
+    -->
+    <!-- Use realsense2_description macro with measured transformation -->
+    <!--
+    IMPORTANT: The measured transformation matrix is from tool0 to camera_color_optical_frame.
+    But the macro attaches at camera_bottom_screw_frame, so we need to compose transforms.
+    Chain in macro (camera_bottom_screw_frame -> camera_color_optical_frame):
+    - camera_bottom_screw_frame -> camera_link: xyz="0.0106 0.0175 0.0125"
+    - camera_link -> camera_color_frame: xyz="0 0.015 0"
+    - camera_color_frame -> camera_color_optical_frame: rpy="-1.5708 0 -1.5708"
+    To get tool0 -> camera_bottom_screw_frame, we need:
+    T_tool0_to_bottom_screw = T_tool0_to_color_optical * inv(T_bottom_screw_to_color_optical)
+    This requires proper matrix composition. For now, using approximate values.
+    TODO: Calculate exact transform using matrix multiplication
+    -->
+    <xacro:sensor_d435 parent="rh_p12_rn_base" name="camera" use_nominal_extrinsics="true" use_mesh="true">
+      <!--
+      Calculated transform: rh_p12_rn_base -> camera_bottom_screw_frame
+      Composed from:
+      - Measured calibration: tool0 -> camera_color_optical_frame
+      - Inverse of: camera_bottom_screw_frame -> camera_color_optical_frame (from macro)
+      - Accounted for tool0 -> rh_p12_rn_base rotation (90° around Z)
+      -->
+      <origin rpy="-1.292395 -1.516365 1.320174" xyz="-0.050732 -0.007579 0.060014"/>
+    </xacro:sensor_d435>
   </xacro:macro>
 </robot>

Commit message: update: add gripper to moveit planning

File: ur_elpis_control/urdf/my_robot_cell_controlled.urdf.xacro (robot description, xacro)
@@ -48,24 +48,3 @@
     headless_mode="$(arg headless_mode)"
   />
-  <!--Gripper ros2_control configuration-->
-  <!-- Note: Gripper control is currently handled via the /control_gripper service.
-       To enable ros2_control for the gripper, a custom hardware interface plugin
-       that wraps the gripper library (librh_p12_rna.so) would need to be created.
-       For now, the gripper joints are defined as revolute in the URDF for visualization
-       but are controlled via the service interface. -->
-  <!--
-  <ros2_control name="gripper" type="actuator">
-    <hardware>
-      <plugin>gripper_hardware/GripperHardwareInterface</plugin>
-    </hardware>
-    <joint name="rh_p12_rn">
-      <command_interface name="position">
-        <param name="min">0.0</param>
-        <param name="max">1.12</param>
-      </command_interface>
-      <state_interface name="position"/>
-      <state_interface name="velocity"/>
-    </joint>
-  </ros2_control>
-  -->
 </robot>

Commit message: update: minor modifications

File: ur_elpis_control/urdf/my_robot_cell_controlled.urdf.xacro (robot description, xacro)
@@ -13,4 +13,5 @@
   <xacro:arg name="physical_params" default="$(find ur_elpis_control)/config/$(arg ur_type)/physical_parameters.yaml"/>
   <xacro:arg name="visual_params" default="$(find ur_elpis_control)/config/$(arg ur_type)/visual_parameters.yaml"/>
+  <!-- Update robot_ip according to your setup-->
   <xacro:arg name="robot_ip" default="192.168.0.100"/>
   <xacro:arg name="headless_mode" default="false" />

File: ur_elpis_description/urdf/my_robot_cell_macro.xacro (robot description, xacro)
@@ -13,34 +13,4 @@
     ">
     <!-- ============================================ -->
-    <!-- Table (Lab Scene) -->
-    <!-- ============================================ -->
-    <joint name="world_to_table" type="fixed">
-      <xacro:insert_block name="origin" />
-      <parent link="${parent}" />
-      <child link="table_base" />
-    </joint>
-    <link name="table_base">
-      <visual>
-        <origin xyz="0 0 0" rpy="0 0 1.5708"/>  <!-- 90 degrees rotation around Z axis -->
-        <geometry>
-          <mesh filename="package://ur_elpis_description/assets/lab_scene/lab_scene.obj"/>
-        </geometry>
-        <material name="table_material">
-          <color rgba="0.7 0.7 0.7 1.0"/>
-        </material>
-      </visual>
-      <collision>
-        <origin xyz="0 0 0" rpy="0 0 1.5708"/>
-        <geometry>
-          <mesh filename="package://ur_elpis_description/assets/lab_scene/lab_scene_vhacd.stl"/>
-        </geometry>
-      </collision>
-      <inertial>
-        <mass value="50.0"/>
-        <origin xyz="0 0 0" rpy="0 0 0"/>
-        <inertia ixx="10.0" ixy="0.0" ixz="0.0" iyy="10.0" iyz="0.0" izz="10.0"/>
-      </inertial>
-    </link>
-    <!-- ============================================ -->
     <!-- Mounting Plate -->
     <!-- ============================================ -->
@@ -67,38 +37,9 @@
       </inertial>
     </link>
-    <joint name="table_to_plate" type="fixed">
-      <parent link="table_base"/>
+    <joint name="world_to_plate" type="fixed">
+      <xacro:insert_block name="origin" />
+      <parent link="${parent}" />
       <child link="mounting_plate"/>
-      <origin xyz="0.0055 0.5 0.7" rpy="0 0 0"/>  <!-- Plate on top of table -->
-    </joint>
-    <!-- ============================================ -->
-    <!-- Ceiling Slab (Height Limiter) -->
-    <!-- ============================================ -->
-    <link name="ceiling_slab">
-      <visual>
-        <geometry>
-          <box size="1.524 1.524 0.05"/>  <!-- Full table dimensions, 5cm thick -->
-        </geometry>
-        <origin xyz="0 0 0" rpy="0 0 0"/>
-        <material name="ceiling_material">
-          <color rgba="0.3 0.3 0.3 0.8"/>  <!-- Semi-transparent dark gray -->
-        </material>
-      </visual>
-      <collision>
-        <geometry>
-          <box size="1.524 1.524 0.05"/>
-        </geometry>
-        <origin xyz="0 0 0" rpy="0 0 0"/>
-      </collision>
-      <inertial>
-        <mass value="20.0"/>
-        <origin xyz="0 0 0" rpy="0 0 0"/>
-        <inertia ixx="4.0" ixy="0.0" ixz="0.0" iyy="4.0" iyz="0.0" izz="4.0"/>
-      </inertial>
-    </link>
-    <joint name="table_to_ceiling" type="fixed">
-      <parent link="table_base"/>
-      <child link="ceiling_slab"/>
-      <origin xyz="0.0 0.0 1.65" rpy="0 0 0"/>  <!-- 0.7m (table top) + 0.95m = 1.65m above table base -->
+      <origin xyz="0.0 0.0 0.0" rpy="0 0 0"/>
     </joint>
     <!-- ============================================ -->
@@ -113,7 +54,6 @@
       physical_parameters_file="${physical_parameters_file}"
       visual_parameters_file="${visual_parameters_file}"
-      generate_ros2_control_tag="false"
-    >
-      <origin xyz="0 0 0" rpy="0 0 -3.141592653589793" />  <!-- Rotate 180 degrees to match original -->
+      generate_ros2_control_tag="false">
+      <origin xyz="0 0 0" rpy="0 0 -3.141592653589793" />   <!-- Rotate 180 degrees to match original config in our lab setup-->
     </xacro:ur_robot>
     <!-- ============================================ -->
@@ -123,5 +63,5 @@
       <color rgba="0.2 0.2 0.2 1.0"/>
     </material>
-    <joint name="tool0_rh_p12_rn_base" type="fixed">
+    <joint name="tool0_rh_p12_rn_base" type="fixed">    <!-- Joint connecting UR tool frame to gripper -->
       <origin rpy="0 0 1.570794" xyz="0 0 0"/>
       <parent link="${ur_type}_tool0"/>
@@ -275,46 +215,11 @@
     <!-- ============================================ -->
     <!-- Using realsense2_description macro for D435 camera -->
-    <!-- Camera transformation from tool0 to camera_color_frame (measured):
-         Matrix:
-         0.99825    -0.027368   -0.052507   -0.007395
-         0.028123    0.99951     0.013702   -0.051154
-         0.052107   -0.015155    0.99853     0.069229
-         0           0           0           1
-         Translation: x=-0.007395, y=-0.051154, z=0.069229
-         Rotation (RPY): roll=-0.01517, pitch=-0.05212, yaw=0.02815
-    -->
-    <!-- Old manual camera definition (commented out):
-    <material name="white">
-      <color rgba="1.0 1.0 1.0 1.0"/>
-    </material>
-    <joint name="d435_joint" type="fixed">
-      <origin rpy="0 -1.5707963267948966 0" xyz="-0.03 0 0.03"/>
-      <parent link="rh_p12_rn_base"/>
-      <child link="d435_bottom_screw_frame"/>
-    </joint>
-    ... (all the manual camera links and joints)
-    -->
-    <!-- Use realsense2_description macro with measured transformation -->
-    <!--
-    IMPORTANT: The measured transformation matrix is from tool0 to camera_color_optical_frame.
-    But the macro attaches at camera_bottom_screw_frame, so we need to compose transforms.
-    Chain in macro (camera_bottom_screw_frame -> camera_color_optical_frame):
-    - camera_bottom_screw_frame -> camera_link: xyz="0.0106 0.0175 0.0125"
-    - camera_link -> camera_color_frame: xyz="0 0.015 0"
-    - camera_color_frame -> camera_color_optical_frame: rpy="-1.5708 0 -1.5708"
-    To get tool0 -> camera_bottom_screw_frame, we need:
-    T_tool0_to_bottom_screw = T_tool0_to_color_optical * inv(T_bottom_screw_to_color_optical)
-    This requires proper matrix composition. For now, using approximate values.
-    TODO: Calculate exact transform using matrix multiplication
-    -->
     <xacro:sensor_d435 parent="rh_p12_rn_base" name="camera" use_nominal_extrinsics="true" use_mesh="true">
-      <!--
-      Calculated transform: rh_p12_rn_base -> camera_bottom_screw_frame
-      Composed from:
-      - Measured calibration: tool0 -> camera_color_optical_frame
-      - Inverse of: camera_bottom_screw_frame -> camera_color_optical_frame (from macro)
-      - Accounted for tool0 -> rh_p12_rn_base rotation (90° around Z)
-      -->
+      <!-- TODO: Calculate exact transform from tool0 to camera_color_optical_frame and replace current values-->
+      <!-- - Measured calibration: tool0 -> camera_color_optical_frame -->
+      <!-- - Inverse of: camera_bottom_screw_frame -> camera_color_optical_frame (from macro) -->
+      <!-- - Accounted for tool0 -> rh_p12_rn_base rotation (90° around Z) -->
       <origin rpy="-1.292395 -1.516365 1.320174" xyz="-0.050732 -0.007579 0.060014"/>
+       <!-- Assuming camera mounted on camera_bottom_screw_frame, so getting accurate pose of camera_bottom_screw_frame is crucial-->
     </xacro:sensor_d435>
   </xacro:macro>
